Commit message: navigation stack working to a degree but gets stuck sometimes.

File: src/ballpicker/urdf/ballpicker.urdf (robot description, URDF)
Before this commit: robot ballpicker, 11 links, 10 joints
Links:
- removed link LM_Wheel
- removed link RM_Wheel
Joints:
- removed joint LM_Wheel_Cont
- removed joint RM_Wheel_Cont

Commit message: new config for navigation stack yet im convinced the robot is incapable of traversing the map comfortably. new design on the way.

File: src/ballpicker/urdf/ballpicker.urdf (robot description, URDF)
Before this commit: robot ballpicker, 9 links, 8 joints
Links:
- link Car_link: mass 19.7238702389369 -> 5.0

Commit message: new robot design working with great navigation functionality

File: src/ballpicker/urdf/ballpicker.urdf (robot description, URDF)
Before this commit: robot ballpicker, 9 links, 8 joints
Links:
- removed link LB_Wheel
- removed link RB_Wheel
- link Car_link: mass 5.0 -> 1.4917848461152376505; geometry collision mesh filename=package://ballpicker/meshes2/car_link.stl; visual mesh filename=package://ballpicker/meshes2/car_link.stl
- link Claw_Left: mass 0.234822404065573 -> 0.077433187135448430793; geometry collision mesh filename=package://ballpicker/meshes2/left_claw.stl; visual mesh filename=package://ballpicker/meshes2/left_claw.stl
- link Claw_Right: mass 0.234822404065573 -> 0.077433187135449055294; geometry collision mesh filename=package://ballpicker/meshes2/right_claw.stl; visual mesh filename=package://ballpicker/meshes2/right_claw.stl
- link LF_Wheel: mass 0.0351748276981348 -> 0.03207771713809098868; geometry collision mesh filename=package://ballpicker/meshes2/p30_isp_a001_3d.stl; collision mesh filename=package://ballpicker/meshes2/pr16_a01_tire_2.stl
- link RF_Wheel: mass 0.0351748276980535 -> 0.03207771713809098868; geometry collision mesh filename=package://ballpicker/meshes2/p30_isp_a001_3d.stl; collision mesh filename=package://ballpicker/meshes2/pr16_a01_tire_2.stl
Joints:
- removed joint LB_Wheel_Cont
- removed joint RB_Wheel_Cont
- joint Claw_Left_J: axis 0 1 0 -> 0 0 1; limit lower=-3.14 upper=3.14 effort=1000 velocity=1 -> effort=1 velocity=20; origin xyz=0.09652 -0.015018 0.17203 rpy=0 0 0 -> xyz=0.0049999999999998240297 -0.10400000000000014788 0.050000000000000169309 rpy=3.141592653589793116 -3.9580907866572562926e-16 3.0015673980571331292
- joint Claw_Right_J: axis 0 1 0 -> 0 0 1; limit lower=-3.14 upper=3.14 effort=1000 velocity=1 -> effort=1 velocity=20; origin xyz=0.08952 -0.015018 0.17203 rpy=0 0 0 -> xyz=-0.0050000000000001952605 -0.10400000000000012013 0.047500000000000167089 rpy=-3.1415926535897926719 -5.9913170964877163588e-16 3.128025583921072883
- joint LF_Wheel_Cont: axis 1 0 0 -> 0 0 -1; limit (none) -> effort=1 velocity=20; origin xyz=0.21777 -0.029518 0.071531 rpy=0 0 0 -> xyz=0.078500000000000166867 -0.034000000000000030198 0.02500000000000004996 rpy=-1.570796326794896558 1.4312143091539777373 1.5707963267948978903
- joint RF_Wheel_Cont: axis 1 0 0 -> 0 0 1; limit (none) -> effort=1 velocity=20; origin xyz=-0.03173 -0.029518 0.071531 rpy=0 0 0 -> xyz=-0.078500000000000291767 -0.034000000000000044076 0.02500000000000004996 rpy=-1.570796326794896558 1.0543435529566484998 -1.57079632679489678
- joint base_to_car: origin xyz=0 -0.09 0 rpy=1.57 0 1.57 -> xyz=0 0.00 0 rpy=0 0 1.57
- joint hokuyo_joint: origin xyz=0.1 0.01 0 rpy=-1.57 0 0 -> xyz=0 0.0 0.15 rpy=0 0 0

Commit message: We now have a method of detecting the balls and transferring their coordinates into the world frame, next well attempt to use this information to control the robot to pick up the balls.

File: src/ballpicker/urdf/ballpicker.urdf (robot description, URDF)
Before this commit: robot ballpicker, 7 links, 6 joints
Links:
- added link kinnect_link, mass 1e-5; collision box size=0.01 0.01 0.01; visual box size=0.01 0.01 0.01
Joints:
- added joint kinnect_joint: type fixed, parent Car_link, child kinnect_link, origin xyz=0 -0.078 0.115 rpy=0 0 -1.57, axis 0 1 0
